File: LED Tuning Board/LED Tuning Board.sch (KiCad schematic (older format))
At the start: 44 parts, among them J4 R_SEL, J5 R_SEL, J6 B_SEL, M1 Mounting, M2 Mounting, M3 Mounting, M4 Mounting, U2 Test Socket

Commit message: Added layout
Parts:
- removed M1, M2, M3, M4: Mounting, mounting:M3_pin, symbol mounting:Mounting
- J4, J6: footprint (none) -> Connector_PinHeader_2.54mm:PinHeader_2x08_P2.54mm_Vertical
- J5: value R_SEL -> G_SEL; footprint (none) -> Connector_PinHeader_2.54mm:PinHeader_2x08_P2.54mm_Vertical
- JP1, JP3, JP4: footprint (none) -> Connector_PinHeader_2.54mm:PinHeader_1x03_P2.54mm_Vertical
- JP2, JP5, JP6: footprint (none) -> Connector_PinHeader_2.54mm:PinHeader_1x02_P2.54mm_Vertical
- R10, R11, R12, R13, R14, R15, R16, R17, R18, R19, R20, R21, R22, R23, R24, R25, R26, R27, R28, R5, R6, R7, R8, R9: footprint (none) -> resistor:R_Axial_DIN0207_L6.3mm_D2.5mm_P10.16mm_Horizontal
- TP3, TP4, TP5, TP6, TP7, TP8: footprint (none) -> testpoint:TestPoint
